File: 3-LSM6DS33-Gyro-Sensor/3.kicad_sch (KiCad schematic)
At the start: 4 parts, among them U1 LSM6DS3

Commit message: schematics
Connections:
- net at U1.13 (SCL): now also A1.32 (SCL/A5)
- net at U1.14 (SDA): now also A1.31 (SDA/A4)
Changed lines of the file:
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@@
+    (stroke (width 0) (type default))
+  )
+  (wire (pts (xy 130.81 93.98) (xy 130.81 99.06))
     (stroke (width 0) (type default))
   )
@@
     (stroke (width 0) (type default))
   )
+  (wire (pts (xy 130.81 99.06) (xy 121.92 99.06))
+    (stroke (width 0) (type default))
+  )
   (wire (pts (xy 153.67 110.49) (xy 153.67 104.14))
     (stroke (width 0) (type default))
   )
+  (wire (pts (xy 127 91.44) (xy 127 96.52))
+    (stroke (width 0) (type default))
+  )
+  (wire (pts (xy 127 96.52) (xy 121.92 96.52))
+    (stroke (width 0) (type default))
+  )
   (wire (pts (xy 129.54 87.63) (xy 129.54 110.49))
+    (stroke (width 0) (type default))
+  )
+  (wire (pts (xy 138.43 91.44) (xy 127 91.44))
+    (stroke (width 0) (type default))
+  )
+  (wire (pts (xy 138.43 93.98) (xy 130.81 93.98))
     (stroke (width 0) (type default))
   )
@@
     (pin "2")
     (instances
-      (project "3.1"
+      (project "3"
         (path "/dd2ddbfe-a4f0-41d0-9010-b4fc27a9d7ce"
           (reference "D1") (unit 1)
@@
     (pin "9")
     (instances
-      (project "3.1"
+      (project "3"
         (path "/dd2ddbfe-a4f0-41d0-9010-b4fc27a9d7ce"
           (reference "U1") (unit 1)
@@
     (pin "2")
     (instances
-      (project "3.1"
+      (project "3"
         (path "/dd2ddbfe-a4f0-41d0-9010-b4fc27a9d7ce"
           (reference "R1") (unit 1)
@@
     (pin "9")
     (instances
-      (project "3.1"
+      (project "3"
         (path "/dd2ddbfe-a4f0-41d0-9010-b4fc27a9d7ce"
           (reference "A1") (unit 1)
